File: quadcopter.sch (EAGLE design)
At the start: 66 parts, among them J1 AVR_SPI_PRG_6NS, Q1 N-CHANNEL_MOSFET, Q2 N-CHANNEL_MOSFET, Q3 N-CHANNEL_MOSFET, Q4 N-CHANNEL_MOSFET, SW2 PUSHBUTTON_SMD-VERTICAL-1, U1 ATMEGA128RFA1

Commit message: Fix gnd/bat_gnd issue and re ran cam job
Connections:
- net BAT_GND: now also C23.1
- net GND: no longer C23.1
Changed lines of the file:
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@@
 <?xml version="1.0" encoding="utf-8"?>
 <!DOCTYPE eagle SYSTEM "eagle.dtd">
-<eagle version="8.2.0">
+<eagle version="8.1.1">
 <drawing>
 <settings>
@@
 <part name="C23" library="quadparts_prebuilt" deviceset="CAPACITOR-NP_" device="SMD-2012-0805_CERAMIC-1UF" value="1uF"/>
 <part name="C24" library="quadparts_prebuilt" deviceset="CAPACITOR-NP_" device="SMD-2012-0805_CERAMIC-1UF" value="1uF"/>
-<part name="GND35" library="quadparts_prebuilt" deviceset="GND" device=""/>
 <part name="GND36" library="quadparts_prebuilt" deviceset="GND" device=""/>
 <part name="J2" library="quadparts-nick" deviceset="MALE_HEADER_2POS" device="-2X1-0.1IN"/>
@@
 <part name="SW2" library="quadparts_prebuilt" deviceset="PUSHBUTTON_" device="SMD-VERTICAL-1"/>
 <part name="GND42" library="quadparts_prebuilt" deviceset="GND" device=""/>
+<part name="GND35" library="quadparts_prebuilt" deviceset="BAT_GND" device=""/>
 </parts>
 <sheets>
@@
 <instance part="C23" gate="G$1" x="-129.54" y="38.1"/>
 <instance part="C24" gate="G$1" x="-91.44" y="27.94"/>
-<instance part="GND35" gate="1" x="-149.86" y="38.1"/>
 <instance part="GND36" gate="1" x="-91.44" y="17.78"/>
 <instance part="J2" gate="G$1" x="-119.38" y="-15.24" rot="R90"/>
@@
 <instance part="SW2" gate="G$1" x="-10.16" y="-129.54"/>
 <instance part="GND42" gate="1" x="2.54" y="-142.24"/>
+<instance part="GND35" gate="1" x="-149.86" y="38.1"/>
 </instances>
 <busses>
@@
 <wire x1="-99.06" y1="20.32" x2="-96.52" y2="20.32" width="0.1524" layer="91"/>
 <wire x1="-96.52" y1="20.32" x2="-96.52" y2="12.7" width="0.1524" layer="91"/>
-</segment>
-<segment>
-<pinref part="C23" gate="G$1" pin="1"/>
-<pinref part="GND35" gate="1" pin="GND"/>
-<wire x1="-129.54" y1="40.64" x2="-149.86" y2="40.64" width="0.1524" layer="91"/>
 </segment>
 <segment>
@@
 <pinref part="GND40" gate="1" pin="BAT_GND"/>
 </segment>
-</net>
+<segment>
+<pinref part="C23" gate="G$1" pin="1"/>
+<wire x1="-129.54" y1="40.64" x2="-149.86" y2="40.64" width="0.1524" layer="91"/>
+<pinref part="GND35" gate="1" pin="BAT_GND"/>
+</segment>
+</net>
